File: HardWare/Electro/Olivia_control/v0.2/v0.2.kicad_sch (KiCad schematic)
At the start: 49 parts, among them J1 PROG, J10 Motor_B, J11 I2C, J12 DAC, J13 UART2, J14 TRIAC OUT_A, J15 TRIAC OUT_B, J16 220V IN, J17 In12V, J2 Input1, J3 Input2, J4 Input3, J5 Input4, J6 LED, J7 Reset, J8 SPI, J9 Motor_A, Q1 BTA16-800B, Q2 BTA16-800B, U1 ESP32-WROOM-32D, U2 MOC3041M, U3 MOC3041M, U4 4N25, U5 AMS1117-3.3, U6 HW-613

Commit message: Add BOM file with updated component configuration
- Added bill-of-materials.csv for v0.2 hardware
- Updated KiCad project settings for BOM export
- Excluded test points from BOM output

🤖 Generated with [Claude Code](https://claude.ai/code)

Co-Authored-By: Claude <noreply@anthropic.com>
Parts:
- PS1, U5: now left out of the parts list
Changed lines of the file:
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@@
 		(unit 1)
 		(exclude_from_sim no)
-		(in_bom yes)
+		(in_bom no)
 		(on_board yes)
 		(dnp no)
@@
 		(unit 1)
 		(exclude_from_sim no)
-		(in_bom yes)
-		(on_board yes)
-		(dnp no)
+		(in_bom no)
+		(on_board yes)
+		(dnp no)
