File: HardWare/Electro/Olivia_control/v0.2/v0.2.kicad_pcb (KiCad board)
At the start: 2 copper layers, 90 x 100 mm, 51 parts, among them J1 PROG, J10 Motor_B, J11 I2C, J12 DAC, J13 UART2, J14 TRIAC OUT_A, J15 TRIAC OUT_B, J16 220V IN, J17 Input 12Vcc max, J2 Input1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

Commit message: replaced 4N25 with TLP181
Parts:
- J17: value Input 12Vcc max -> In12V
- U4: value 4N25 -> TLP181; footprint Package_DIP:SMDIP-6_W9.53mm -> Package_SO:SOIC-4_4.55x3.7mm_P2.54mm
- moved U4 1.69 mm to (73.8, 126.8)
Connections:
- U4 pad 3: unconnected-(U4-NC-Pad3) -> Net-(BR1-Pad-)
- U4 pad 6: unconnected-(U4-Pad6) -> /ZERO
Routing:
- net Net-(BR1-Pad-): track 7.79 -> 9.56 mm
- net /ZERO: track 59.5 -> 58.1 mm
